Commit message: Add collision counter: dual-sim abstraction (Ignition + Isaac Sim contract)
- navlearn_msgs: add collision_count to TrajectoryMetric.msg (Safety metrics section)
- bumperbot_description: add contact sensor (type=contact, 50 Hz) on base_link for Ignition
- collision_monitor (new node): subscribes to ros_gz_interfaces/msg/Contacts via
  ros_gz_bridge, performs rising-edge detection, publishes std_msgs/Empty to
  /navlearn/collision — one message per collision event
- trajectory_metric: subscribes to /navlearn/collision; resets collision_count_ on
  episode START; increments on each Empty msg while active; sets msg_.collision_count
  in publishReport()
- metrics_compiler: adds Collision Count CSV column, total_collisions + collisions_per_goal
  to JSON run summary
- benchmarks.launch.py: adds ros_gz_bridge (parameter_bridge) for contact sensor topic
  with world_name substitution, and launches collision_monitor node
- trajectory_metric.yaml: documents collision_topic and ground truth dual-sim contract
  (Isaac Sim: publish TransformStamped to gt_topic via Isaac ROS bridge, no code change
  needed — trajectory_metric already uses a ROS 2 subscription)

Isaac Sim adapter contract: OmniGraph extension publishes std_msgs/Empty to
/navlearn/collision on rising-edge contact (see docs/isaac_sim/ — future work).
trajectory_metric requires zero changes to support Isaac Sim once the topic is live.

Co-Authored-By: Claude Sonnet 4.6 <noreply@anthropic.com>

File: src/bumperbot_description/urdf/bumperbot_gazebo.xacro (robot description, xacro)
@@ -119,4 +119,14 @@
     </sensor>
   </gazebo>
+  <!-- Contact Sensor (Ignition/Fortress) — used by navlearn_benchmarks collision_monitor -->
+  <gazebo reference="base_link">
+    <sensor name="contact_sensor" type="contact">
+      <always_on>true</always_on>
+      <update_rate>50</update_rate>
+      <contact>
+        <collision>base_link_collision</collision>
+      </contact>
+    </sensor>
+  </gazebo>
   <!-- 2D Laser Sensor -->
   <gazebo reference="laser_link">

Commit message: Pivot collision detection to scan-based threshold; remove Ignition Contact system plugin
Contact sensor (Ignition contact-system world plugin) caused ~6 min startup hang due to
mesh collision pre-processing, breaking controller and map frame. Pivot to scan-based
rising-edge detection in trajectory_metric (collision_scan_threshold_m: 0.15 m). Removed
plugin from both world files. Disabled contact sensor block in bumperbot_gazebo.xacro with
explanatory comment. Isaac Sim adapter path preserved via /navlearn/collision topic.

Co-Authored-By: Claude Sonnet 4.6 <noreply@anthropic.com>

File: src/bumperbot_description/urdf/bumperbot_gazebo.xacro (robot description, xacro)
@@ -119,14 +119,10 @@
     </sensor>
   </gazebo>
-  <!-- Contact Sensor (Ignition/Fortress) — used by navlearn_benchmarks collision_monitor -->
-  <gazebo reference="base_link">
-    <sensor name="contact_sensor" type="contact">
-      <always_on>true</always_on>
-      <update_rate>50</update_rate>
-      <contact>
-        <collision>base_link_collision</collision>
-      </contact>
-    </sensor>
-  </gazebo>
+  <!-- Contact Sensor (Ignition/Fortress) — DISABLED.                                          -->
+  <!-- The ignition-gazebo-contact-system world plugin is required for contact sensors to fire, -->
+  <!-- but adding it to the world SDF causes Ignition to pre-process ALL mesh collision        -->
+  <!-- geometry in the scene at startup (~6 min hang → spawn timeout → no controller/map).    -->
+  <!-- Collision counting instead uses scan-based detection in trajectory_metric (threshold    -->
+  <!-- on minimum LiDAR range). See collision_scan_threshold_m in trajectory_metric.yaml.     -->
   <!-- 2D Laser Sensor -->
   <gazebo reference="laser_link">
